Commit message: add moving stick for husky ur5

File: husky/husky_description/urdf/husky.urdf.xacro (robot description, xacro)
@@ -22,8 +22,4 @@
 -->
 <robot name="husky" xmlns:xacro="http://ros.org/wiki/xacro">
-  <xacro:arg name="transmission_hw_interface" default="hardware_interface/PositionJointInterface"/>
-  <xacro:include filename="$(find ur_description)/urdf/ur5.urdf.xacro" />
-  <xacro:include filename="$(find robotiq_ft_sensor)/urdf/robotiq_ft300.urdf.xacro" />
-  <xacro:include filename="$(find robotiq_85_description)/urdf/robotiq_85_gripper.urdf.xacro" />
   <xacro:arg name="laser_enabled" default="$(optenv HUSKY_LMS1XX_ENABLED 0)" />
   <xacro:arg name="laser_xyz" default="$(optenv HUSKY_LMS1XX_XYZ 0.2206 0.0 0.00635)" />
@@ -87,45 +83,4 @@
     </collision>
   </link>
-   <!-- #############################bumper_test###############################-->
-  <link name="bumper_link">
-    <inertial>
-        <origin rpy="0 0 0" xyz="0 0 0"/>
-        <mass value="0.0000000000001"/>
-        <inertia ixx="0.00000001" ixy="0.00000001" ixz="0.00000001" iyy="0.00000001" iyz="0.00000001" izz="0.00000001"/>
-    </inertial>
-    <!-- <visual>
-        <origin rpy="0 0 0" xyz="0 0 0.1"/>
-        <geometry>
-            <box size="1.0 0.7 0.31"/>
-        </geometry>
-        <material name="red">
-            <color rgba="1.0 0.0 0.0 1.0"/>
-        </material>
-    </visual> -->
-    <collision name="base_link_fixed_joint_lump__robot/bumper_link">
-        <origin rpy="0 0 0" xyz="0 0 0.1"/>
-        <geometry>
-            <box size="1.0 0.7 0.31"/>
-        </geometry>
-    </collision>
-  </link>
-  <joint name="bumper_joint" type="fixed">
-      <origin xyz="0 0 0" rpy="0.0 0.0 0.0"/>
-      <parent link="base_link" />
-      <child link="bumper_link" />
-  </joint>
-  <gazebo reference="bumper_link">
-    <sensor name='contactsensor_sensor' type='contact'>
-      <always_on>true</always_on>
-      <updaterate>100.0</updaterate>
-      <contact>
-        <collision>base_link_fixed_joint_lump__robot/bumper_link_collision_2</collision>
-      </contact>
-          <plugin name="gazebo_ros_bumper_controller" filename="libgazebo_ros_bumper.so">
-              <bumperTopicName>bumper_states</bumperTopicName>
-              <frameName>world</frameName>
-          </plugin>
-    </sensor>
-  </gazebo>
   <!-- Base footprint is on the ground under the robot -->
   <link name="base_footprint"/>
@@ -262,126 +217,3 @@
   <!-- Optional for Clearpath internal softwares -->
   <xacro:include filename="$(arg cpr_urdf_extras)" />
-  <link name="stick_link">
-    <inertial>
-      <mass value="50" />
-      <origin xyz="0 0 0" />
-      <inertia ixx="50.0" ixy="0.0" ixz="0.0"
-        iyy="50.0" iyz="0.0"
-        izz="50.0" />
-    </inertial>
-    <visual>
-      <origin xyz="0 0 0" />
-      <geometry>
-        <box size="0 0 0" /> <!-- does not need to match collision -->
-      </geometry>
-    </visual>
-    <collision>
-      <origin xyz="0 0 0" />
-      <geometry>
-        <box size="0 0 0" />
-      </geometry>
-    </collision>
-  </link>
-  <joint name="stick_joint" type="fixed">
-    <parent link="top_plate_link" />
-    <child link = "stick_link" />
-    <origin xyz="0.0 0.0 0" rpy="0.0 0.0 0.0" />
-  </joint>
-  <link name="stick_move_link">
-    <inertial>
-      <mass value="2" />
-      <origin xyz="0 0 0" />
-      <inertia ixx="50.0" ixy="0.0" ixz="0.0"
-        iyy="50.0" iyz="0.0"
-        izz="50.0" />
-    </inertial>
-    <visual>
-      <origin xyz="0 0 0" />
-      <geometry>
-        <box size="0.05 0.09 0.03" /> <!-- does not need to match collision -->
-      </geometry>
-    </visual>
-    <collision>
-      <origin xyz="0 0 0" />
-      <geometry>
-        <box size="0.05 0.09 0.03" />
-      </geometry>
-    </collision>
-  </link>
-  <joint name="stick_move_joint" type="prismatic">
-    <parent link="stick_link" />
-    <child link = "stick_move_link" />
-    <axis xyz="1 0 0" />
-    <limit effort="20000.0" lower="0" upper="0.5" velocity="0.2"/>
-    <origin xyz="0.46 0.11 0.48" rpy="0.0 0.0 0.0" />
-  </joint>
-  <link name="bumper_stick_link">
-      <inertial>
-          <origin rpy="0 0 0" xyz="0 0 0"/>
-          <mass value="0.0000000000001"/>
-          <inertia ixx="0.00000001" ixy="0.00000001" ixz="0.00000001" iyy="0.00000001" iyz="0.00000001" izz="0.00000001"/>
-      </inertial>
-      <!-- <visual>
-          <origin rpy="0 0 0" xyz="0.035 0 0"/>
-          <geometry>
-              <box size="0.005 0.09 0.03"/>
-          </geometry>
-          <material name="red">
-              <color rgba="1.0 0.0 0.0 1.0"/>
-          </material>
-      </visual> -->
-      <collision name="stick_move_link_fixed_joint_lump__/bumper_stick_link">
-          <origin rpy="0 0 0" xyz="0.035 0 0"/>
-          <geometry>
-              <box size="0.005 0.09 0.03"/>
-          </geometry>
-      </collision>
-    </link>
-    <joint name="bumper_stick_joint" type="fixed">
-        <origin xyz="0 0 0" rpy="0.0 0.0 0.0"/>
-        <parent link="stick_move_link" />
-        <child link="bumper_stick_link" />
-    </joint>
-    <gazebo reference="bumper_stick_link">
-      <sensor name='contactsensor_sensor' type='contact'>
-        <always_on>true</always_on>
-        <updaterate>100.0</updaterate>
-        <contact>
-          <collision>stick_move_link_fixed_joint_lump__/bumper_stick_link_collision_1</collision>
-        </contact>
-            <plugin name="gazebo_ros_bumper_controller" filename="libgazebo_ros_bumper.so">
-                <bumperTopicName>bumper_stick_states</bumperTopicName>
-                <frameName>world</frameName>
-            </plugin>
-      </sensor>
-    </gazebo>
-  <transmission name="tran1">
-    <type>transmission_interface/SimpleTransmission</type>
-    <joint name="stick_move_joint">
-      <hardwareInterface>EffortJointInterface</hardwareInterface>
-    </joint>
-    <actuator name="motor1">
-      <hardwareInterface>EffortJointInterface</hardwareInterface>
-      <mechanicalReduction>1</mechanicalReduction>
-    </actuator>
-  </transmission>
-  <xacro:ur5_robot prefix="ur5/" joint_limited="false"
-    transmission_hw_interface="$(arg transmission_hw_interface)"
-  />
-  <joint name="ur5_joint" type="fixed">
-    <parent link="top_plate_link" />
-    <child link = "ur5/base_link" />
-    <origin xyz="0.0 0.0 0.0" rpy="0.0 0.0 0.0" />
-  </joint>
-  <xacro:robotiq_ft300 prefix="" parent="ur5/tool0" >
-        <origin xyz="0 0 0" rpy="0 0 ${-pi/2}"/>
-    </xacro:robotiq_ft300>
-  <xacro:robotiq_85_gripper prefix="" parent="robotiq_ft_frame_id">
-    <origin xyz="0 0 0" rpy="0 ${-pi/2} 0"/>
-  </xacro:robotiq_85_gripper>
-  <!-- lidar -->
-  <xacro:include filename="$(find husky_ur5)/urdf/3d_lidar.urdf.xacro" />
-  <xacro:velodyne_lidar name="front_laser" topic="$(arg robot_namespace)/points" parent="base_link" max_range="75" update_rate="15">
-      <origin xyz="0.45 0.0 0.325" rpy="0 0 0"/>
-  </xacro:velodyne_lidar>
 </robot>

File: husky/husky_description/urdf/husky_stick.urdf.xacro (robot description, xacro)
@@ -22,8 +22,4 @@
 -->
 <robot name="husky" xmlns:xacro="http://ros.org/wiki/xacro">
-  <xacro:arg name="transmission_hw_interface" default="hardware_interface/PositionJointInterface"/>
-  <xacro:include filename="$(find ur_description)/urdf/ur5.urdf.xacro" />
-  <xacro:include filename="$(find robotiq_ft_sensor)/urdf/robotiq_ft300.urdf.xacro" />
-  <xacro:include filename="$(find robotiq_85_description)/urdf/robotiq_85_gripper.urdf.xacro" />
   <xacro:arg name="laser_enabled" default="$(optenv HUSKY_LMS1XX_ENABLED 0)" />
   <xacro:arg name="laser_xyz" default="$(optenv HUSKY_LMS1XX_XYZ 0.2206 0.0 0.00635)" />
@@ -87,5 +83,5 @@
     </collision>
   </link>
-   <!-- #############################bumper_test###############################-->
+  <!-- #############################bumper_test###############################-->
   <link name="bumper_link">
     <inertial>
@@ -262,5 +258,5 @@
   <!-- Optional for Clearpath internal softwares -->
   <xacro:include filename="$(arg cpr_urdf_extras)" />
-  <link name="stick_link">
+   <link name="stick_link">
     <inertial>
       <mass value="50" />
@@ -290,5 +286,5 @@
   <link name="stick_move_link">
     <inertial>
-      <mass value="2" />
+      <mass value="1" />
       <origin xyz="0 0 0" />
       <inertia ixx="50.0" ixy="0.0" ixz="0.0"
@@ -299,5 +295,5 @@
       <origin xyz="0 0 0" />
       <geometry>
-        <box size="0.05 0.09 0.03" /> <!-- does not need to match collision -->
+        <box size="0.5 0.1 0.1" /> <!-- does not need to match collision -->
       </geometry>
     </visual>
@@ -305,5 +301,5 @@
       <origin xyz="0 0 0" />
       <geometry>
-        <box size="0.05 0.09 0.03" />
+        <box size="0.5 0.1 0.1" />
       </geometry>
     </collision>
@@ -313,47 +309,20 @@
     <child link = "stick_move_link" />
     <axis xyz="1 0 0" />
-    <limit effort="20000.0" lower="0" upper="0.5" velocity="0.2"/>
-    <origin xyz="0.46 0.11 0.48" rpy="0.0 0.0 0.0" />
-  </joint>
-  <link name="bumper_stick_link">
-      <inertial>
-          <origin rpy="0 0 0" xyz="0 0 0"/>
-          <mass value="0.0000000000001"/>
-          <inertia ixx="0.00000001" ixy="0.00000001" ixz="0.00000001" iyy="0.00000001" iyz="0.00000001" izz="0.00000001"/>
-      </inertial>
-      <!-- <visual>
-          <origin rpy="0 0 0" xyz="0.035 0 0"/>
-          <geometry>
-              <box size="0.005 0.09 0.03"/>
-          </geometry>
-          <material name="red">
-              <color rgba="1.0 0.0 0.0 1.0"/>
-          </material>
-      </visual> -->
-      <collision name="stick_move_link_fixed_joint_lump__/bumper_stick_link">
-          <origin rpy="0 0 0" xyz="0.035 0 0"/>
-          <geometry>
-              <box size="0.005 0.09 0.03"/>
-          </geometry>
-      </collision>
-    </link>
-    <joint name="bumper_stick_joint" type="fixed">
-        <origin xyz="0 0 0" rpy="0.0 0.0 0.0"/>
-        <parent link="stick_move_link" />
-        <child link="bumper_stick_link" />
-    </joint>
-    <gazebo reference="bumper_stick_link">
-      <sensor name='contactsensor_sensor' type='contact'>
-        <always_on>true</always_on>
-        <updaterate>100.0</updaterate>
-        <contact>
-          <collision>stick_move_link_fixed_joint_lump__/bumper_stick_link_collision_1</collision>
-        </contact>
+    <limit effort="10000.0" lower="0" upper="0.5" velocity="0.2"/>
+    <origin xyz="0.18 0.0 0.4" rpy="0.0 0.0 0.0" />
+  </joint>
+  <!-- <gazebo reference="stick_move_link">
+        <sensor type="contact" name="contactsensor_sensor">
+            <always_on>true</always_on>
+            <updaterate>100.0</updaterate>
+            <contact>
+                <collision>X2/base_link_fixed_joint_lump__X2/chassis_link_collision</collision>
+            </contact>
             <plugin name="gazebo_ros_bumper_controller" filename="libgazebo_ros_bumper.so">
-                <bumperTopicName>bumper_stick_states</bumperTopicName>
+                <bumperTopicName>bumper_stick</bumperTopicName>
                 <frameName>world</frameName>
             </plugin>
-      </sensor>
-    </gazebo>
+        </sensor>
+  </gazebo> -->
   <transmission name="tran1">
     <type>transmission_interface/SimpleTransmission</type>
@@ -366,20 +335,6 @@
     </actuator>
   </transmission>
-  <xacro:ur5_robot prefix="ur5/" joint_limited="false"
-    transmission_hw_interface="$(arg transmission_hw_interface)"
-  />
-  <joint name="ur5_joint" type="fixed">
-    <parent link="top_plate_link" />
-    <child link = "ur5/base_link" />
-    <origin xyz="0.0 0.0 0.0" rpy="0.0 0.0 0.0" />
-  </joint>
-  <xacro:robotiq_ft300 prefix="" parent="ur5/tool0" >
-        <origin xyz="0 0 0" rpy="0 0 ${-pi/2}"/>
-    </xacro:robotiq_ft300>
-  <xacro:robotiq_85_gripper prefix="" parent="robotiq_ft_frame_id">
-    <origin xyz="0 0 0" rpy="0 ${-pi/2} 0"/>
-  </xacro:robotiq_85_gripper>
   <!-- lidar -->
-  <xacro:include filename="$(find husky_ur5)/urdf/3d_lidar.urdf.xacro" />
+  <xacro:include filename="$(find husky_description)/urdf/3d_lidar.urdf.xacro" />
   <xacro:velodyne_lidar name="front_laser" topic="$(arg robot_namespace)/points" parent="base_link" max_range="75" update_rate="15">
       <origin xyz="0.45 0.0 0.325" rpy="0 0 0"/>
