Commit message: modify stick for training

File: husky_ur5/urdf/husky_ur5_contact.urdf.xacro (robot description, xacro)
@@ -313,5 +313,5 @@
     <child link = "stick_move_link" />
     <axis xyz="1 0 0" />
-    <limit effort="20000.0" lower="0" upper="0.5" velocity="0.2"/>
+    <limit effort="50000.0" lower="0" upper="0.5" velocity="1"/>
     <origin xyz="0.46 0.11 0.48" rpy="0.0 0.0 0.0" />
   </joint>

Commit message: stick -> yellow bar

File: husky_ur5/urdf/husky_ur5_contact.urdf.xacro (robot description, xacro)
@@ -299,5 +299,5 @@
       <origin xyz="0 0 0" />
       <geometry>
-        <box size="0.05 0.09 0.03" /> <!-- does not need to match collision -->
+        <box size="1 0.09 0.03" />
       </geometry>
     </visual>
@@ -305,8 +305,11 @@
       <origin xyz="0 0 0" />
       <geometry>
-        <box size="0.05 0.09 0.03" />
-      </geometry>
-    </collision>
-  </link>
+        <box size="1 0.09 0.03" />
+      </geometry>
+    </collision>
+  </link>
+  <gazebo reference="stick_move_link">
+    <material>Gazebo/Yellow</material>
+  </gazebo>
   <joint name="stick_move_joint" type="prismatic">
     <parent link="stick_link" />
@@ -366,5 +369,5 @@
     </actuator>
   </transmission>
-  <xacro:ur5_robot prefix="ur5/" joint_limited="false"
+  <!-- <xacro:ur5_robot prefix="ur5/" joint_limited="false"
     transmission_hw_interface="$(arg transmission_hw_interface)"
   />
@@ -379,5 +382,5 @@
   <xacro:robotiq_85_gripper prefix="" parent="robotiq_ft_frame_id">
     <origin xyz="0 0 0" rpy="0 ${-pi/2} 0"/>
-  </xacro:robotiq_85_gripper>
+  </xacro:robotiq_85_gripper> -->
   <!-- lidar -->
   <xacro:include filename="$(find husky_ur5)/urdf/3d_lidar.urdf.xacro" />

Commit message: sensor modify

File: husky_ur5/urdf/husky_ur5_contact.urdf.xacro (robot description, xacro)
@@ -286,5 +286,5 @@
     <parent link="top_plate_link" />
     <child link = "stick_link" />
-    <origin xyz="0.0 0.0 0" rpy="0.0 0.0 0.0" />
+    <origin xyz="-0.2 0.0 0" rpy="0.0 0.0 0.0" />
   </joint>
   <link name="stick_move_link">
@@ -299,11 +299,11 @@
       <origin xyz="0 0 0" />
       <geometry>
-        <box size="1 0.09 0.03" />
+        <box size="0.5 0.09 0.03" />
       </geometry>
     </visual>
-    <collision>
-      <origin xyz="0 0 0" />
-      <geometry>
-        <box size="1 0.09 0.03" />
+    <collision name="stick_link_fixed_joint_lump__/stick_move_link">
+      <origin xyz="0 0 0" />
+      <geometry>
+        <box size="0.5 0.09 0.03" />
       </geometry>
     </collision>
@@ -319,5 +319,5 @@
     <origin xyz="0.46 0.11 0.48" rpy="0.0 0.0 0.0" />
   </joint>
-  <link name="bumper_stick_link">
+  <!-- <link name="bumper_stick_link">
       <inertial>
           <origin rpy="0 0 0" xyz="0 0 0"/>
@@ -325,5 +325,5 @@
           <inertia ixx="0.00000001" ixy="0.00000001" ixz="0.00000001" iyy="0.00000001" iyz="0.00000001" izz="0.00000001"/>
       </inertial>
-      <!-- <visual>
+      <visual>
           <origin rpy="0 0 0" xyz="0.035 0 0"/>
           <geometry>
@@ -333,5 +333,5 @@
               <color rgba="1.0 0.0 0.0 1.0"/>
           </material>
-      </visual> -->
+      </visual>
       <collision name="stick_move_link_fixed_joint_lump__/bumper_stick_link">
           <origin rpy="0 0 0" xyz="0.035 0 0"/>
@@ -345,11 +345,11 @@
         <parent link="stick_move_link" />
         <child link="bumper_stick_link" />
-    </joint>
-    <gazebo reference="bumper_stick_link">
+    </joint> -->
+    <gazebo reference="stick_move_link">
       <sensor name='contactsensor_sensor' type='contact'>
         <always_on>true</always_on>
         <updaterate>100.0</updaterate>
         <contact>
-          <collision>stick_move_link_fixed_joint_lump__/bumper_stick_link_collision_1</collision>
+          <collision>stick_move_link_fixed_joint_lump__stick_link_fixed_joint_lump__/stick_move_link_collision</collision>
         </contact>
             <plugin name="gazebo_ros_bumper_controller" filename="libgazebo_ros_bumper.so">
@@ -369,22 +369,8 @@
     </actuator>
   </transmission>
-  <!-- <xacro:ur5_robot prefix="ur5/" joint_limited="false"
-    transmission_hw_interface="$(arg transmission_hw_interface)"
-  />
-  <joint name="ur5_joint" type="fixed">
-    <parent link="top_plate_link" />
-    <child link = "ur5/base_link" />
-    <origin xyz="0.0 0.0 0.0" rpy="0.0 0.0 0.0" />
-  </joint>
-  <xacro:robotiq_ft300 prefix="" parent="ur5/tool0" >
-        <origin xyz="0 0 0" rpy="0 0 ${-pi/2}"/>
-    </xacro:robotiq_ft300>
-  <xacro:robotiq_85_gripper prefix="" parent="robotiq_ft_frame_id">
-    <origin xyz="0 0 0" rpy="0 ${-pi/2} 0"/>
-  </xacro:robotiq_85_gripper> -->
   <!-- lidar -->
   <xacro:include filename="$(find husky_ur5)/urdf/3d_lidar.urdf.xacro" />
-  <xacro:velodyne_lidar name="front_laser" topic="$(arg robot_namespace)/points" parent="base_link" max_range="75" update_rate="15">
-      <origin xyz="0.45 0.0 0.325" rpy="0 0 0"/>
+  <xacro:velodyne_lidar name="front_laser" topic="$(arg robot_namespace)/points" parent="top_plate_link" max_range="75" update_rate="15">
+      <origin xyz="0.0 0.0 0.25" rpy="0 0 0"/>
   </xacro:velodyne_lidar>
 </robot>

Commit message: fix bugs

File: husky_ur5/urdf/husky_ur5_contact.urdf.xacro (robot description, xacro)
@@ -310,34 +310,4 @@
     <origin xyz="0.46 0.11 0.48" rpy="0.0 0.0 0.0" />
   </joint>
-<<<<<<< HEAD
-  <!-- <link name="bumper_stick_link">
-      <inertial>
-          <origin rpy="0 0 0" xyz="0 0 0"/>
-          <mass value="0.0000000000001"/>
-          <inertia ixx="0.00000001" ixy="0.00000001" ixz="0.00000001" iyy="0.00000001" iyz="0.00000001" izz="0.00000001"/>
-      </inertial>
-      <visual>
-          <origin rpy="0 0 0" xyz="0.035 0 0"/>
-          <geometry>
-              <box size="0.005 0.09 0.03"/>
-          </geometry>
-          <material name="red">
-              <color rgba="1.0 0.0 0.0 1.0"/>
-          </material>
-      </visual>
-      <collision name="stick_move_link_fixed_joint_lump__/bumper_stick_link">
-          <origin rpy="0 0 0" xyz="0.035 0 0"/>
-          <geometry>
-              <box size="0.005 0.09 0.03"/>
-          </geometry>
-      </collision>
-    </link>
-    <joint name="bumper_stick_joint" type="fixed">
-        <origin xyz="0 0 0" rpy="0.0 0.0 0.0"/>
-        <parent link="stick_move_link" />
-        <child link="bumper_stick_link" />
-    </joint> -->
-=======
->>>>>>> upstream/main
     <gazebo reference="stick_move_link">
       <sensor name='contactsensor_sensor' type='contact'>
